File: shinsanwaswitch_PCB/shinsanwaswitch_v1.1/shinsanwaswitch_v1.1-standard.kicad_pcb (KiCad board)
At the start: 2 copper layers, 26.3 x 15.4 mm, 9 parts, among them J1 Conn_01x05_Male, Q1 2SC5395

Commit message: Update shinsanwaswitch_v1.1-standard.kicad_pcb
Parts:
- STI1: moved to F.Cu
Changed lines of the file:
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@@
+    )
+  )
+  (footprint "Diode_SMD:D_SOD-123" (layer "F.Cu")
+    (at 131.71 75.99 180)
+    (descr "SOD-123")
+    (tags "SOD-123")
+    (property "Имя листа" "")
+    (property "Файл листа" "C:/Users/steel/Desktop/shinsanwaswitchplusleddriver_rpi-352/shinsanwaswitch.kicad_sch")
+    (attr smd)
+    (fp_text reference "STI1" (at 2.96 -0.05 90) (layer "F.SilkS")
+      (effects (font (size 0.8 0.8) (thickness 0.15)))
+    )
+    (fp_text value "NSI45020AT1G" (at 0 2.1) (layer "F.Fab")
+      (effects (font (size 1 1) (thickness 0.15)))
+    )
+    (fp_text user "${REFERENCE}" (at 0 -2) (layer "F.Fab")
+      (effects (font (size 1 1) (thickness 0.15)))
+    )
+    (fp_line (start -2.25 -1) (end 1.65 -1) (layer "F.SilkS") (width 0.12))
+    (fp_line (start -2.25 -1) (end -2.25 1) (layer "F.SilkS") (width 0.12))
+    (fp_line (start -2.25 1) (end 1.65 1) (layer "F.SilkS") (width 0.12))
+    (fp_line (start 2.35 -1.15) (end 2.35 1.15) (layer "F.CrtYd") (width 0.05))
+    (fp_line (start -2.35 -1.15) (end 2.35 -1.15) (layer "F.CrtYd") (width 0.05))
+    (fp_line (start 2.35 1.15) (end -2.35 1.15) (layer "F.CrtYd") (width 0.05))
+    (fp_line (start -2.35 -1.15) (end -2.35 1.15) (layer "F.CrtYd") (width 0.05))
+    (fp_line (start -0.75 0) (end -0.35 0) (layer "F.Fab") (width 0.1))
+    (fp_line (start 0.25 -0.4) (end 0.25 0.4) (layer "F.Fab") (width 0.1))
+    (fp_line (start -0.35 0) (end -0.35 -0.55) (layer "F.Fab") (width 0.1))
+    (fp_line (start -0.35 0) (end -0.35 0.55) (layer "F.Fab") (width 0.1))
+    (fp_line (start 1.4 -0.9) (end 1.4 0.9) (layer "F.Fab") (width 0.1))
+    (fp_line (start 0.25 0) (end 0.75 0) (layer "F.Fab") (width 0.1))
+    (fp_line (start -1.4 0.9) (end -1.4 -0.9) (layer "F.Fab") (width 0.1))
+    (fp_line (start -0.35 0) (end 0.25 -0.4) (layer "F.Fab") (width 0.1))
+    (fp_line (start 1.4 0.9) (end -1.4 0.9) (layer "F.Fab") (width 0.1))
+    (fp_line (start 0.25 0.4) (end -0.35 0) (layer "F.Fab") (width 0.1))
+    (fp_line (start -1.4 -0.9) (end 1.4 -0.9) (layer "F.Fab") (width 0.1))
+    (pad "1" smd rect locked (at -1.65 0 180) (size 0.9 1.2) (layers "F.Cu" "F.Paste" "F.Mask")
+      (net 2 "Net-(D1-Pad1)"))
+    (pad "2" smd rect locked (at 1.65 0 180) (size 0.9 1.2) (layers "F.Cu" "F.Paste" "F.Mask")
+      (net 6 "/+12V"))
+    (model "${KISYS3DMOD}/Diode_SMD.3dshapes/D_SOD-123.wrl"
+      (offset (xyz 0 0 0))
+      (scale (xyz 1 1 1))
+      (rotate (xyz 0 0 0))
     )
   )
@@
     )
   )
-  (footprint "Diode_SMD:D_SOD-123" (layer "B.Cu")
-    (at 131.71 75.99 180)
-    (descr "SOD-123")
-    (tags "SOD-123")
-    (property "Имя листа" "")
-    (property "Файл листа" "C:/Users/steel/Desktop/shinsanwaswitchplusleddriver_rpi-352/shinsanwaswitch.kicad_sch")
-    (attr smd)
-    (fp_text reference "STI1" (at 2.96 0.05 90) (layer "B.SilkS")
-      (effects (font (size 0.8 0.8) (thickness 0.15)) (justify mirror))
-    )
-    (fp_text value "NSI45020AT1G" (at 0 -2.1 180) (layer "B.Fab")
-      (effects (font (size 1 1) (thickness 0.15)) (justify mirror))
-    )
-    (fp_text user "${REFERENCE}" (at 0 2 180) (layer "B.Fab")
-      (effects (font (size 1 1) (thickness 0.15)) (justify mirror))
-    )
-    (fp_line (start -2.25 1) (end 1.65 1) (layer "B.SilkS") (width 0.12))
-    (fp_line (start -2.25 1) (end -2.25 -1) (layer "B.SilkS") (width 0.12))
-    (fp_line (start -2.25 -1) (end 1.65 -1) (layer "B.SilkS") (width 0.12))
-    (fp_line (start 2.35 1.15) (end 2.35 -1.15) (layer "B.CrtYd") (width 0.05))
-    (fp_line (start -2.35 1.15) (end 2.35 1.15) (layer "B.CrtYd") (width 0.05))
-    (fp_line (start 2.35 -1.15) (end -2.35 -1.15) (layer "B.CrtYd") (width 0.05))
-    (fp_line (start -2.35 1.15) (end -2.35 -1.15) (layer "B.CrtYd") (width 0.05))
-    (fp_line (start -0.75 0) (end -0.35 0) (layer "B.Fab") (width 0.1))
-    (fp_line (start 0.25 0.4) (end 0.25 -0.4) (layer "B.Fab") (width 0.1))
-    (fp_line (start -0.35 0) (end -0.35 0.55) (layer "B.Fab") (width 0.1))
-    (fp_line (start -0.35 0) (end -0.35 -0.55) (layer "B.Fab") (width 0.1))
-    (fp_line (start 1.4 0.9) (end 1.4 -0.9) (layer "B.Fab") (width 0.1))
-    (fp_line (start 0.25 0) (end 0.75 0) (layer "B.Fab") (width 0.1))
-    (fp_line (start -1.4 -0.9) (end -1.4 0.9) (layer "B.Fab") (width 0.1))
-    (fp_line (start -0.35 0) (end 0.25 0.4) (layer "B.Fab") (width 0.1))
-    (fp_line (start 1.4 -0.9) (end -1.4 -0.9) (layer "B.Fab") (width 0.1))
-    (fp_line (start 0.25 -0.4) (end -0.35 0) (layer "B.Fab") (width 0.1))
-    (fp_line (start -1.4 0.9) (end 1.4 0.9) (layer "B.Fab") (width 0.1))
-    (pad "1" smd rect locked (at -1.65 0 180) (size 0.9 1.2) (layers "B.Cu" "B.Paste" "B.Mask")
-      (net 2 "Net-(D1-Pad1)"))
-    (pad "2" smd rect locked (at 1.65 0 180) (size 0.9 1.2) (layers "B.Cu" "B.Paste" "B.Mask")
-      (net 6 "/+12V"))
-    (model "${KISYS3DMOD}/Diode_SMD.3dshapes/D_SOD-123.wrl"
-      (offset (xyz 0 0 0))
-      (scale (xyz 1 1 1))
-      (rotate (xyz 0 0 0))
-    )
-  )
   (gr_line (start 135.175 88.425) (end 131.725 88.425) (layer "F.SilkS") (width 0.12))
   (gr_line (start 135.25 84.425) (end 131.7 84.425) (layer "F.SilkS") (width 0.12))
@@
   (segment (start 152.27 86.2) (end 151.145 87.325) (width 0.7) (layer "B.Cu") (net 1))
   (segment (start 142.895 88.625) (end 142.9 88.63) (width 0.7) (layer "B.Cu") (net 1))
-  (segment (start 133.36 75.99) (end 133.920888 75.99) (width 0.8) (layer "B.Cu") (net 2))
-  (segment (start 133.920888 75.99) (end 135.015048 77.08416) (width 0.8) (layer "B.Cu") (net 2))
+  (segment (start 133.36 75.99) (end 133.920888 75.99) (width 0.8) (layer "F.Cu") (net 2))
+  (segment (start 133.920888 75.99) (end 135.015048 77.08416) (width 0.8) (layer "F.Cu") (net 2))
   (segment (start 145.265299 88.621846) (end 147.191846 88.621846) (width 1) (layer "B.Cu") (net 3))
   (segment (start 152.27 88.7) (end 153.525 87.445) (width 0.4) (layer "B.Cu") (net 4))
@@
   (segment (start 133.009629 85.019999) (end 139.709999 85.019999) (width 0.4) (layer "B.Cu") (net 5))
   (segment (start 139.709999 85.019999) (end 140.775 86.085) (width 0.4) (layer "B.Cu") (net 5))
-  (segment (start 130.05 78.35) (end 130.05 77.470372) (width 0.8) (layer "B.Cu") (net 6))
-  (segment (start 132.304628 79.725) (end 131.425 79.725) (width 0.8) (layer "B.Cu") (net 6))
-  (segment (start 130.05 75.99) (end 130.05 77.470372) (width 0.8) (layer "B.Cu") (net 6))
-  (segment (start 131.425 79.725) (end 130.05 78.35) (width 0.8) (layer "B.Cu") (net 6))
-  (segment (start 134.25 81.725) (end 135.015048 80.959952) (width 0.8) (layer "B.Cu") (net 7))
-  (segment (start 135.015048 80.959952) (end 135.015048 79.08416) (width 0.8) (layer "B.Cu") (net 7))
-  (segment (start 132.304628 81.725) (end 134.25 81.725) (width 0.8) (layer "B.Cu") (net 7))
+  (segment (start 130.05 78.35) (end 130.05 77.470372) (width 0.8) (layer "F.Cu") (net 6))
+  (segment (start 132.304628 79.725) (end 131.425 79.725) (width 0.8) (layer "F.Cu") (net 6))
+  (segment (start 130.05 75.99) (end 130.05 77.470372) (width 0.8) (layer "F.Cu") (net 6))
+  (segment (start 131.425 79.725) (end 130.05 78.35) (width 0.8) (layer "F.Cu") (net 6))
+  (segment (start 134.25 81.725) (end 135.015048 80.959952) (width 0.8) (layer "F.Cu") (net 7))
+  (segment (start 135.015048 80.959952) (end 135.015048 79.08416) (width 0.8) (layer "F.Cu") (net 7))
+  (segment (start 132.304628 81.725) (end 134.25 81.725) (width 0.8) (layer "F.Cu") (net 7))
   (segment (start 137.47 83.72) (end 139.365 81.825) (width 0.8) (layer "B.Cu") (net 8))
   (segment (start 133.62 83.72) (end 133.615 83.725) (width 0.8) (layer "B.Cu") (net 8))

Commit message: Update shinsanwaswitch_v1.1-standard.kicad_pcb
Other:
- board text added: "SHINSANWASWITCH board by steelpuxnastik / Doctopus from ProjectDIVA.net ver 1.1 with LED Driver 2020"
- board text removed: "SHINSANWASWITCH board by steelpuxnastik / Doctopus from ProjectDIVA.net ver 1.0 with LED Driver 2020"
Changed lines of the file:
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@@
     (effects (font (size 0.5 0.5) (thickness 0.125)) (justify mirror))
   )
-  (gr_text "SHINSANWASWITCH board\nby steelpuxnastik / Doctopus\nfrom ProjectDIVA.net\nver 1.0 with LED Driver\n2020" (at 147.75 80.425) (layer "B.SilkS")
+  (gr_text "SHINSANWASWITCH board\nby steelpuxnastik / Doctopus\nfrom ProjectDIVA.net\nver 1.1 with LED Driver\n2020" (at 147.75 80.425) (layer "B.SilkS")
     (effects (font (size 0.5 0.5) (thickness 0.1)) (justify mirror))
   )
