File: shinsanwaswitch_PCB/shinsanwaswitch_v1.1-LEDDriver_one-layer.kicad_sch (KiCad schematic)
At the start: 9 parts, among them J1 Conn_01x05_Male, Q1 2SC5395

Commit message: Massive update of DIY-boards to make it easier to print and drill
Parts:
- PC1: footprint RPI-221:RPI-352 -> RPI-221:RPI-352_otherholes
Changed lines of the file:
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@@
     (property "Reference" "PC1" (id 0) (at 138 68.6226 0))
     (property "Value" "RPI-352" (id 1) (at 138 70.9215 0))
-    (property "Footprint" "RPI-221:RPI-352" (id 2) (at 131.5466 83.8708 0)
+    (property "Footprint" "RPI-221:RPI-352_otherholes" (id 2) (at 131.5466 83.8708 0)
       (effects (font (size 1.27 1.27) italic) (justify left) hide)
     )
@@
     )
     (path "/e1c04423-3561-4ccd-94dd-ce73aeebcd59"
-      (reference "PC1") (unit 1) (value "RPI-352") (footprint "RPI-221:RPI-352")
+      (reference "PC1") (unit 1) (value "RPI-352") (footprint "RPI-221:RPI-352_otherholes")
     )
     (path "/bee2bef6-3a14-4cbf-8e61-794bd3a2d0e3"
